Commit message: Add files via upload

File: kinova_files/gen3_version2.urdf (robot description, URDF)
Before this commit: robot gen3, 8 links, 7 joints
Links:
- added link gripper_link
Joints:
- added joint joint__gripper: type fixed, parent bracelet_link, child gripper_link, origin xyz=0 0 -0.16 rpy=0 0 0
- joint joint_1: limit lower=-2.41 upper=2.41 effort=39 velocity=1.3963 -> lower=-6.28 upper=6.28 effort=39 velocity=1.3963

Commit message: Add files via upload

File: kinova_files/gen3_version2.urdf (robot description, URDF)
Before this commit: robot gen3, 9 links, 8 joints
Joints:
- removed joint joint__gripper
- added joint joint_gripper: type fixed, parent bracelet_link, child gripper_link, origin xyz=0 0 -0.10 rpy=0 0 0
- joint joint_1: origin xyz=0 0 0.15643 rpy=3.1416 2.7629E-18 -4.9305E-36 -> xyz=0 0 0.015643 rpy=3.1416 2.7629E-18 -4.9305E-36
- joint joint_3: limit lower=-2.41 upper=2.41 effort=39 velocity=1.3963 -> lower=-6.28 upper=6.28 effort=39 velocity=1.3963
- joint joint_5: limit lower=-2.41 upper=2.41 effort=9 velocity=1.2218 -> lower=-6.28 upper=6.28 effort=39 velocity=1.3963
- joint joint_7: limit lower=-2.41 upper=2.41 effort=9 velocity=1.2218 -> lower=-6.28 upper=6.28 effort=39 velocity=1.3963
